File: HW/Sequencer_Button_Matrix_sch.kicad_sch (KiCad schematic)
At the start: 10 parts, among them IC1 74LS138

Commit message: Pin remapping, connect AVCC, filtering, TP
Connections:
- net BUTTON_IN renamed STEP_IN
Changed lines of the file:
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@@
 		)
 	)
-	(global_label "BUTTON_IN"
+	(global_label "STEP_IN"
 		(shape input)
 		(at 86.36 86.36 270)
@@
 		)
 		(property "Intersheetrefs" "${INTERSHEET_REFS}"
-			(at 86.36 99.4448 90)
-			(hide yes)
-			(show_name no)
-			(do_not_autoplace no)
-			(effects
-				(font
-					(size 1.27 1.27)
-				)
-				(justify right)
-			)
-		)
-	)
-	(global_label "BUTTON_IN"
+			(at 86.36 96.8442 90)
+			(hide yes)
+			(show_name no)
+			(do_not_autoplace no)
+			(effects
+				(font
+					(size 1.27 1.27)
+				)
+				(justify right)
+			)
+		)
+	)
+	(global_label "STEP_IN"
 		(shape input)
 		(at 152.4 86.36 270)
@@
 		)
 		(property "Intersheetrefs" "${INTERSHEET_REFS}"
-			(at 152.4 99.4448 90)
-			(hide yes)
-			(show_name no)
-			(do_not_autoplace no)
-			(effects
-				(font
-					(size 1.27 1.27)
-				)
-				(justify right)
-			)
-		)
-	)
-	(global_label "BUTTON_IN"
+			(at 152.4 96.8442 90)
+			(hide yes)
+			(show_name no)
+			(do_not_autoplace no)
+			(effects
+				(font
+					(size 1.27 1.27)
+				)
+				(justify right)
+			)
+		)
+	)
+	(global_label "STEP_IN"
 		(shape input)
 		(at 53.34 86.36 270)
@@
 		)
 		(property "Intersheetrefs" "${INTERSHEET_REFS}"
-			(at 53.34 99.4448 90)
+			(at 53.34 96.8442 90)
 			(hide yes)
 			(show_name no)
@@
 		)
 	)
-	(global_label "BUTTON_IN"
+	(global_label "STEP_IN"
 		(shape input)
 		(at 20.32 86.36 270)
@@
 		)
 		(property "Intersheetrefs" "${INTERSHEET_REFS}"
-			(at 20.32 99.4448 90)
-			(hide yes)
-			(show_name no)
-			(do_not_autoplace no)
-			(effects
-				(font
-					(size 1.27 1.27)
-				)
-				(justify right)
-			)
-		)
-	)
-	(global_label "BUTTON_IN"
+			(at 20.32 96.8442 90)
+			(hide yes)
+			(show_name no)
+			(do_not_autoplace no)
+			(effects
+				(font
+					(size 1.27 1.27)
+				)
+				(justify right)
+			)
+		)
+	)
+	(global_label "STEP_IN"
 		(shape input)
 		(at 218.44 86.36 270)
@@
 		)
 		(property "Intersheetrefs" "${INTERSHEET_REFS}"
-			(at 218.44 99.4448 90)
+			(at 218.44 96.8442 90)
 			(hide yes)
 			(show_name no)
@@
 		)
 	)
-	(global_label "BUTTON_IN"
+	(global_label "STEP_IN"
 		(shape input)
 		(at 251.46 86.36 270)
@@
 		)
 		(property "Intersheetrefs" "${INTERSHEET_REFS}"
-			(at 251.46 99.4448 90)
+			(at 251.46 96.8442 90)
 			(hide yes)
 			(show_name no)
@@
 		)
 	)
-	(global_label "BUTTON_IN"
+	(global_label "STEP_IN"
 		(shape input)
 		(at 185.42 86.36 270)
@@
 		)
 		(property "Intersheetrefs" "${INTERSHEET_REFS}"
-			(at 185.42 99.4448 90)
+			(at 185.42 96.8442 90)
 			(hide yes)
 			(show_name no)
@@
 		)
 	)
-	(global_label "BUTTON_IN"
+	(global_label "STEP_IN"
 		(shape input)
 		(at 119.38 86.36 270)
@@
 		)
 		(property "Intersheetrefs" "${INTERSHEET_REFS}"
-			(at 119.38 99.4448 90)
-			(hide yes)
-			(show_name no)
+			(at 119.38 96.8442 90)
+			(hide yes)
+			(show_name no)
