File: HW/melodiasekvensseri.kicad_pcb (KiCad board)
At the start: 2 copper layers, 60.6 x 110 mm, 50 parts, among them IC1 74LS138, J1 Conn_02x05_Odd_Even, J2 Clock_In, J3 Gate_Out, J4 CV_Out, J5 Conn_02x03_Odd_Even, J6 Conn_01x04, U1 TLV2372IP

Commit message: Pin remapping, connect AVCC, filtering, TP
Parts:
- added C14: 100n, Capacitor_THT:C_Disc_D5.0mm_W2.5mm_P5.00mm, B.Cu at (151.0, 100.7)
- added R8: 10, Resistor_THT:R_Axial_DIN0207_L6.3mm_D2.5mm_P10.16mm_Horizontal, B.Cu at (156.2, 97.7)
- added TP_12V1: TestPoint, TestPoint:TestPoint_Pad_2.0x2.0mm, F.Cu at (165.6, 55.2)
- added TP_A5V1: TestPoint, TestPoint:TestPoint_Pad_2.0x2.0mm, F.Cu at (159.7, 122.7)
- added TP_AGND1: TestPoint, TestPoint:TestPoint_Pad_2.0x2.0mm, F.Cu at (175.9, 134.7)
- added TP_D5V1: TestPoint, TestPoint:TestPoint_Pad_2.0x2.0mm, F.Cu at (165.5, 82.6)
- added TP_DAC_OUT1: TestPoint, TestPoint:TestPoint_Pad_2.0x2.0mm, F.Cu at (159.7, 127.1)
- added TP_DGND1: TestPoint, TestPoint:TestPoint_Pad_2.0x2.0mm, F.Cu at (175.2, 96.3)
- moved J5 8.55 mm to (157.9, 93.6)
- moved C13 4.45 mm to (151.6, 93.8), turned to 180 degrees
- moved J6 4.21 mm to (140.1, 74.6)
- moved C11 1.10 mm to (148.6, 59.1)
- moved C12 1.10 mm to (155.7, 59.1)
- moved RE1 1.10 mm to (147.5, 55.8)
- moved R3 1.10 mm to (135.9, 58.1)
- moved REG2 0.87 mm to (162.4, 98.8)
Connections:
- J6 pad 1: TXD -> RXD
- J6 pad 2: RXD -> TXD
- MC1 pad 11: DEMUX_C -> STEP_IN
- MC1 pad 12: DEMUX_B -> DEMUX_A
- MC1 pad 13: DEMUX_A -> DEMUX_B
- MC1 pad 14: CLK_IN -> DEMUX_C
- MC1 pad 20: unconnected-(MC1-AVCC-Pad20) -> Net-(MC1-AVCC)
- MC1 pad 26: BUTTON_IN -> ENC_B
- MC1 pad 4: ENC_B -> ENC_A
- MC1 pad 5: ENC_A -> CLK_IN
- S1 pad 4: BUTTON_IN -> STEP_IN
- S2 pad 4: BUTTON_IN -> STEP_IN
- S3 pad 4: BUTTON_IN -> STEP_IN
- S4 pad 4: BUTTON_IN -> STEP_IN
- S5 pad 4: BUTTON_IN -> STEP_IN
- S6 pad 4: BUTTON_IN -> STEP_IN
- S7 pad 4: BUTTON_IN -> STEP_IN
- S8 pad 4: BUTTON_IN -> STEP_IN
Routing:
- net STEP_IN: track 0.00 -> 173.8 mm
- net BUTTON_IN: track 124.9 -> 0.00 mm, vias 10 -> 0
- net D_+5V: track 198.8 -> 230.2 mm, vias 2 -> 0
- net CLK_IN: track 64.2 -> 85.3 mm
- net Net-(DAC1-VOUT): track 8.25 -> 25.2 mm
- net DEMUX_C: track 44.5 -> 30.6 mm
- net ENC_B: track 51.2 -> 37.9 mm
- net SPI_SCK: track 29.2 -> 42.3 mm
- net SPI_MOSI: track 29.7 -> 41.4 mm, vias 4 -> 2
- net DEMUX_B: track 40.5 -> 31.0 mm
- net SPI_MISO: track 11.8 -> 19.3 mm
- net A_+5V: track 51.8 -> 58.8 mm
- net Net-(MC1-AVCC): track 0.00 -> 5.66 mm
- net RXD: track 15.8 -> 10.8 mm
- net ENC_A: track 42.6 -> 37.8 mm
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Other:
- board text added: "Melody Sequencer JSi, JHa, LHo 2026"
